File: gate-opener.kicad_sch (KiCad schematic)
At the start: 0 parts

Commit message: schematic init
Parts:
- added J1: Screw_Terminal_01x04_5.08mm, TerminalBlock:TerminalBlock_bornier-4_P5.08mm, symbol Connector:Screw_Terminal_01x04
- added J2, J3: Screw_Terminal_01x02_5.08mm, TerminalBlock:TerminalBlock_bornier-2_P5.08mm, symbol Connector:Screw_Terminal_01x02
- added J4, J5: BK-18650-PC4, jannett_footprints:BK-18650-PC4_MPD, symbol Connector_Generic:Conn_02x02_Counter_Clockwise
- added K1: DPDT Relay, Relay_THT:Relay_DPDT_Kemet_EC2_NU, symbol Relay:EC2-3NU
- added M1: Motor_DC, symbol Motor:Motor_DC
- added PS1: 24V DC/DC, Converter_DCDC:Converter_DCDC_XP_POWER-ITXxxxxSA_THT, symbol Converter_DCDC:ITX2403SA
- added Q1: MMBT3904, Package_TO_SOT_SMD:SOT-23, symbol Transistor_BJT:MMBT3904
- added U1: ESP32 Dev Board, jannett_footprints:ESP32_MODULE, symbol jannett_symbols:ESP32_Module
Connections:
- new net: J3.2 (Pin_2), K1.1, Q1.3 (C)
- new net: K1.10, K1.5, PS1.6 (+Vout)
- new net: J3.1 (Pin_1), K1.12
- new net: K1.3, K1.8, PS1.7 (-Vout)
- new net: K1.4, M1.1 (+)
- new net: K1.9, M1.2 (-)
- new net: J4.1 (Pin_1), J4.3 (Pin_3)
- new net: J4.2 (Pin_2), J5.4 (Pin_4)
- new net: J2.2 (Pin_2), PS1.1 (-Vin)
- new net: J2.1 (Pin_1), PS1.2 (+Vin)
- new net: J5.1 (Pin_1), J5.3 (Pin_3)
- new net GND: J4.4 (Pin_4), Q1.2 (E)
Other:
- note added: "10V-16V Input, 24V output Boost Converter Module"
- note added: "Linear Actuator"
- note added: "NOT ON BOARD: REPRESENTATION ONLY"
- note added: "Relay Coil"

Commit message: schematic
Parts:
- added D1, D2: 1N4004, Diode_THT:D_DO-41_SOD81_P10.16mm_Horizontal, symbol Diode:1N4004
- added Q10, Q2, Q3, Q4, Q5: AOD403, Package_TO_SOT_SMD:TO-252-2, symbol Transistor_FET:QM6015D
- added Q6, Q7, Q8, Q9: MMBT3904, Package_TO_SOT_SMD:SOT-23, symbol Transistor_BJT:MMBT3904
- added R1, R2, R3, R4: 100, Resistor_SMD:R_2512_6332Metric_Pad1.40x3.35mm_HandSolder, symbol Device:R_US
- added R10, R5, R6, R8: 100K, Resistor_SMD:R_0603_1608Metric_Pad0.98x0.95mm_HandSolder, symbol Device:R_US
- added R11, R12, R7, R9: 10K, Resistor_SMD:R_0603_1608Metric_Pad0.98x0.95mm_HandSolder, symbol Device:R_US
Connections:
- net GND: now also J2.2 (Pin_2), PS1.1 (-Vin), D1.2 (A), Q6.2 (E), Q7.2 (E), Q8.2 (E), Q9.2 (E), R1.2
- net at J3.2 (Pin_2), K1.1, Q1.3 (C): now also D2.2 (A)
- net at J3.1 (Pin_1), K1.12: now also D2.1 (K)
- net VBAT_MID1: now reaches J4.1 (Pin_1), J4.3 (Pin_3)
- net VBAT_MID1: now also Q2.3 (S), R2.2, R5.1
- net VBAT_MID2: now reaches J4.2 (Pin_2), J5.4 (Pin_4)
- net VBAT_MID2: now also Q3.3 (S), R3.2, R6.1
- net at J2.1 (Pin_1), PS1.2 (+Vin): now also D1.1 (K), Q10.2 (D)
- net VBAT_MID3: now reaches J5.1 (Pin_1), J5.3 (Pin_3)
- net VBAT_MID3: now also Q4.3 (S), R4.2, R8.1
- net VBAT: now reaches J5.2 (Pin_2)
- net VBAT: now also Q5.3 (S), R10.1
- new net: Q9.1 (B), R12.1
- new net: Q2.1 (G), Q9.3 (C), R5.2
- new net: Q4.1 (G), Q7.3 (C), R8.2
- new net: Q4.2 (D), R3.1
- new net: Q5.2 (D), R4.1
- new net: Q5.1 (G), Q8.3 (C), R10.2
- new net: Q6.1 (B), R7.1
- new net: Q3.1 (G), Q6.3 (C), R6.2
- new net: Q2.2 (D), R1.1
- new net: Q7.1 (B), R9.1
- new net: Q3.2 (D), R2.1
- new net: Q8.1 (B), R11.1
Other:
- moved on the sheet: J4, J5, U1

Commit message: schematic
Parts:
- added J6: Screw_Terminal_01x04_5.08mm, TerminalBlock:TerminalBlock_bornier-4_P5.08mm, symbol Connector:Screw_Terminal_01x04
- added R14: 0.1, Resistor_SMD:R_Shunt_Vishay_WSK2512_6332Metric_T2.21mm, symbol Device:R_Shunt_US
Connections:
- net GND: now also J1.2 (Pin_2), J1.4 (Pin_4), R14.4
- net VBAT: now also Q10.3 (S)
- net +24V: now reaches J1.3 (Pin_3)
- net +24V: now also J6.2 (Pin_2), J6.3 (Pin_3)
- new net: J6.1 (Pin_1), J6.4 (Pin_4), R14.1
Other:
- note added: "Add in sense resistor on the negative leads so that we can see if the motor stalls"
- note added: "Change out because I need the 24V on board to drive the relay"
- note added: "I like Gemini's idea, change this out for an ESP32-S2 dev board"
- note added: "It has 2 DAC's and better ADC's, and better low power mode."
- note added: "to DPDT Relay poles"
- moved on the sheet: U1

Commit message: schematic
Parts:
- removed Q2, Q3, Q4, Q5: AOD403, Package_TO_SOT_SMD:TO-252-2, symbol Transistor_FET:QM6015D
- removed Q6, Q7, Q8, Q9: MMBT3904, Package_TO_SOT_SMD:SOT-23, symbol Transistor_BJT:MMBT3904
- removed R1: 100, Resistor_SMD:R_2512_6332Metric_Pad1.40x3.35mm_HandSolder, symbol Device:R_US
- added C1, C13, C2, C3, C4, C5, C6, C7, C8: 0.1uF, Capacitor_SMD:C_0603_1608Metric_Pad1.08x0.95mm_HandSolder, symbol Device:C_Small
- added C10: 4.7uF, Capacitor_SMD:C_0603_1608Metric_Pad1.08x0.95mm_HandSolder, symbol Device:C_Small
- added C11, C9: 1uF, Capacitor_SMD:C_0603_1608Metric_Pad1.08x0.95mm_HandSolder, symbol Device:C_Small
- added C12: 10uF, Capacitor_SMD:C_0603_1608Metric_Pad1.08x0.95mm_HandSolder, symbol Device:C_Small
- added J7, J8: 53048-0610, Connector_Molex:Molex_PicoBlade_53048-0610_1x06_P1.25mm_Horizontal, symbol Connector_Generic:Conn_01x06
- added R1: 0.1, Resistor_SMD:R_Shunt_Vishay_WSK2512_6332Metric_T2.21mm, symbol Device:R_Shunt_US
- added R13, R15, R16: 10K, Resistor_SMD:R_0603_1608Metric_Pad0.98x0.95mm_HandSolder, symbol Device:R_US
- added SW1: TL3305BF260QG, Button_Switch_SMD:SW_SPST_TL3305B, symbol Switch:SW_Push
- added TH1, TH2, TH3: 10K, Resistor_THT:R_Axial_DIN0204_L3.6mm_D1.6mm_P2.54mm_Vertical, symbol Device:Thermistor_US
- added U2: BQ7692006PWR, Package_SO:TSSOP-20_4.4x6.5mm_P0.65mm, symbol Battery_Management:BQ76920PW
- R10: value 100K -> 10K
- R2, R3, R4: footprint Resistor_SMD:R_2512_6332Metric_Pad1.40x3.35mm_HandSolder -> Resistor_SMD:R_0603_1608Metric_Pad0.98x0.95mm_HandSolder
- R5, R6, R8: value 100K -> 100
- R7, R9: value 10K -> 100
Connections:
- net GND: now also R10.2, U1.2 (GND), U1.29 (GND), C10.2, C11.2, C12.2, C13.2, C2.2, C3.1, C4.1, C5.2, C9.2, J7.4 (Pin_4), J8.4 (Pin_4), R1.4, TH1.2, TH2.2, TH3.2, U2.3 (VSS); no longer J4.4 (Pin_4)
- net VBAT: now also R4.2, R9.1, C9.1, U2.9 (REGSRC); no longer R10.1
- net THERM2: now reaches R12.1
- net THERM2: now also TH3.1
- net VC0: now reaches R5.2
- net VC0: now also C4.2, U2.17 (VC0)
- net VC34: now reaches R8.2
- net VC34: now also C7.1, C8.2, U2.13 (VC4), U2.14 (VC3)
- net at R3.1: now also R1.2
- net BAT: now reaches R4.1
- net BAT: now also C12.1, U2.10 (BAT)
- net CELL2: now reaches R7.1
- net CELL2: now also J4.2 (Pin_2), J5.4 (Pin_4)
- net VC1: now reaches R6.2
- net VC1: now also C5.1, C6.2, SW1.2, U2.16 (VC1)
- net VC5: now reaches R9.2
- net VC5: now also C8.1, U2.12 (VC5)
- net at R2.1: now also R1.3
- net TS1: now reaches R11.1
- net TS1: now also C13.1, TH1.1, U2.6 (TS1)
- net at R11.2: now also SW1.1
- net +3.3V: now reaches U1.1 (+3.3V)
- net +3.3V: now also R12.2, R13.2, R15.1, R16.1
- net +5V: now reaches U1.30 (VIN)
- net +5V: now also J7.1 (Pin_1), J8.1 (Pin_1)
- net VC2: now reaches R7.2
- net VC2: now also C6.1, C7.2, U2.15 (VC2)
- net VBAT_MID1 renamed CELL1
- net CELL1: now also R6.1; no longer R2.2, R5.1
- removed net VBAT_MID2: J4.2 (Pin_2), J5.4 (Pin_4), R3.2, R6.1
- net VBAT_MID3 renamed CELL3
- net CELL3: no longer R4.2
- new net: J8.5 (Pin_5), R16.2
- new net: J7.5 (Pin_5), R15.2
- new net: R10.1, U2.20 (ALERT)
- new net: C11.1, U2.7 (CAP1)
- new net CELL0: J4.4 (Pin_4), R1.1, R5.1
- new net I2C_SCL: U2.5 (SCL)
- new net I2C_SDA: U2.4 (SDA)
- new net LIDAR_RX1: J7.2 (Pin_2)
- new net LIDAR_RX2: J8.2 (Pin_2)
- new net LIDAR_TX1: J7.3 (Pin_3)
- new net LIDAR_TX2: J8.3 (Pin_3)
- new net REGOUT: C10.1, U2.8 (REGOUT)
- new net SRN: C1.1, C3.2, R3.2, U2.19 (SRN)
- new net SRP: C1.2, C2.1, R2.2, U2.18 (SRP)
- new net THERM1: R13.1, TH2.1
- no-connect marks 0 -> 4
Other:
- note added: "I2C Addr = 0x18"
- note added: "TF-Luna LIDAR"
- note added: "Table 9-2"
- moved on the sheet: J4, J5, U1

Commit message: schematic
Parts:
- removed U1: ESP32 Dev Board, jannett_footprints:ESP32_MODULE, symbol jannett_symbols:ESP32_Module
- added J10, J9: Conn_02x08_Odd_Even, symbol Connector_Generic:Conn_02x08_Odd_Even
Connections:
- net +3.3V: now also J10.1 (Pin_1)
- net +5V: now also J9.2 (Pin_2)
- net GND: now also J9.3 (Pin_3), J9.4 (Pin_4)
- new net EN: J10.15 (Pin_15)
Other:
- note added: "ESP32 S2 Mini"

Commit message: schematic
Parts:
- removed J2, J3: Screw_Terminal_01x02_5.08mm, TerminalBlock:TerminalBlock_bornier-2_P5.08mm, symbol Connector:Screw_Terminal_01x02
- added J2: Screw_Terminal_01x04_5.08mm, TerminalBlock:TerminalBlock_bornier-4_P5.08mm, symbol Connector:Screw_Terminal_01x04
- added Q2: MMBT3904, Package_TO_SOT_SMD:SOT-23, symbol Transistor_BJT:MMBT3904
- added R17: 1K, Resistor_SMD:R_0603_1608Metric_Pad0.98x0.95mm_HandSolder, symbol Device:R_US
- added R18, R19: 10K, Resistor_SMD:R_0603_1608Metric_Pad0.98x0.95mm_HandSolder, symbol Device:R_US
Connections:
- net +24V: now also D2.1 (K), J2.3 (Pin_3)
- net GND: now also Q2.2 (E); no longer PS1.1 (-Vin)
- net VBAT: now also R19.2
- net at Q10.1 (G): now also Q2.3 (C), R19.1
- net BOOST_PWR: now reaches D1.1 (K), Q10.2 (D)
- net BOOST_PWR: now also J1.1 (Pin_1); no longer PS1.2 (+Vin)
- net at K1.12: no longer D2.1 (K)
- net at D2.2 (A), Q1.3 (C): now also J2.4 (Pin_4); no longer K1.1
- net at Q1.1 (B): now also R17.2
- net RTN: now reaches J6.1 (Pin_1), J6.4 (Pin_4), R14.1
- new net: Q2.1 (B), R18.2
- new net BOOST_EN: R18.1
- new net DIR: R17.1
- now unconnected: K1.10, K1.3, K1.5, K1.8, PS1.6 (+Vout), PS1.7 (-Vout)
Other:
- note added: "ADD: 5V Buck converter"
- note added: "ADD: Current amp"
- note added: "ADD: E-STOP Button circuit (comparator and protection)"
- note added: "ADD: Solar input and measurements"
- note added: "ADD: indicator LEDs"
- note removed: "Add in sense resistor on the negative leads so that we can see if the motor stalls"
- note removed: "Change out because I need the 24V on board to drive the relay"
- moved on the sheet: D1, D2, J1, J10, J6, J7, J8, J9, K1, M1, Q1, Q10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

Commit message: schematic
Parts:
- added C14, C20: 0.1uF, Capacitor_SMD:C_0603_1608Metric_Pad1.08x0.95mm_HandSolder, symbol Device:C_Small
- added C15, C18: 100uF, Capacitor_SMD:CP_Elec_6.3x5.4_Nichicon, symbol Device:C_Polarized_Small_US
- added C19, C22: 22uF, Capacitor_SMD:C_1210_3225Metric_Pad1.33x2.70mm_HandSolder, symbol Device:C_Small
- added C21: 4.7uF, Capacitor_SMD:C_0603_1608Metric_Pad1.08x0.95mm_HandSolder, symbol Device:C_Small
- added D3: 1N5819WS, Diode_SMD:D_SOD-323_HandSoldering, symbol Diode:1N5819WS
- added H1, H2, H3, H4: MountingHole, MountingHole:MountingHole_3.2mm_M3, symbol Mechanical:MountingHole
- added L1: 56uH, Inductor_SMD:L_Chilisin_BWVS00606045, symbol Device:L
- added Q3, Q4: QM6006D, Package_TO_SOT_SMD:TO-252-2, symbol Transistor_FET:QM6006D
- added R20: 2K, Resistor_SMD:R_0603_1608Metric_Pad0.98x0.95mm_HandSolder, symbol Device:R_US
- added R23: 10.5K, Resistor_SMD:R_0603_1608Metric_Pad0.98x0.95mm_HandSolder, symbol Device:R_US
- added TP10, TP3, TP5, TP6, TP7, TP8, TP9: 5016, Jarrett_Footprint_Library:TestPoint_Keystone_5016_Compact, symbol Connector:TestPoint
- added U1: RT8110BGJ8, Package_TO_SOT_SMD:SOT-23-8_Handsoldering, symbol 1Jarrett_Symbol_Library:RT8110BGJ8
Connections:
- net +5V: now also C15.1, C22.1, L1.2, R23.2, TP3.1
- net GND: now also C14.2, C15.2, C18.2, C19.2, C21.2, C22.2, Q4.3 (S), R20.2, TP5.1, TP6.1, U1.3 (GND)
- net VBAT: now also C14.1, C18.1, C19.1, Q3.2 (D), U1.7 (VIN)
- new net: R20.1, R23.1, TP10.1, U1.8 (FB)
- new net: Q4.1 (G), TP9.1, U1.2 (LGATE)
- new net: C20.2, L1.1, Q3.3 (S), Q4.2 (D), U1.6 (PHASE)
- new net: C21.1, D3.1 (K), TP7.1, U1.1 (VCC)
- new net: Q3.1 (G), U1.4 (UGATE)
- new net: C20.1, D3.2 (A), TP8.1, U1.5 (BOOT)
Other:
- note removed: "ADD: 5V Buck converter"
